File: LED_Cube.brd (EAGLE design)
At the start: 100 x 80 mm, 35 parts, among them IC1 MSGEQ7SOIC, Q1 16MHz, U1 ATMEGA328P-AU, U2 TLC5940PWP, U3 TLC5940PWP, X1 1503_02

Commit message: schematic 80%/board 25%
Parts:
- moved SV3 98.4 mm to (4.06, 20.8)
- moved SV1 97.8 mm to (14.7, 3.30), turned to 180 degrees
- moved U3 79.7 mm to (17.8, 12.2), turned to 90 degrees
- moved R5 69.9 mm to (17.8, 18.3), turned to 90 degrees
- moved U2 68.3 mm to (40.9, 12.4), turned to 90 degrees
- moved SV2 67.6 mm to (38.4, 3.05), turned to 0 degrees
- moved JP3 62.2 mm to (5.33, 48.5), turned to 270 degrees
- moved R4 58.3 mm to (37.3, 18.8), turned to 90 degrees
- moved JP1 55.1 mm to (36.8, 76.2), turned to 0 degrees
- moved Q4 44.6 mm to (25.4, 58.9), turned to 0 degrees
- moved JP4 40.6 mm to (6.86, 39.4), turned to 90 degrees
- moved Q2 38.4 mm to (37.3, 58.9), turned to 0 degrees
- moved Q3 38.2 mm to (48.5, 58.9), turned to 0 degrees
- moved C13 36.3 mm to (14.5, 18.5), turned to 90 degrees
- moved C4 35.8 mm to (9.40, 39.1), turned to 90 degrees
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Connections:
- net LAYER2_OFF: now also Q3.G; no longer Q2.G
- net LAYER3_OFF: now also Q2.G; no longer Q3.G
Routing:
- net +5V: track 16.4 -> 95.3 mm
- net SPI_MISO: track 0.00 -> 26.7 mm
- net LAYER1_OFF: track 37.3 -> 11.0 mm
- net SPI_SCLK: track 0.00 -> 26.2 mm
- net MSG_RST: track 0.00 -> 23.2 mm
- net N$36: track 17.9 -> 38.9 mm
- net SPI_MOSI: track 0.00 -> 20.4 mm, vias 0 -> 2
- net N$42: track 9.94 -> 29.3 mm
- net N$43: track 7.93 -> 27.3 mm
- net N$6: track 16.7 -> 0.00 mm
- net N$4: track 15.1 -> 0.00 mm
- net LAYER3_OFF: track 0.00 -> 14.7 mm
- net MSG_STROBE: track 0.00 -> 14.6 mm
- net N$1: track 10.5 -> 0.00 mm
- net LAYER2_OFF: track 33.1 -> 24.9 mm
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Other:
- board size 100 x 80 mm -> 61.9 x 80 mm

Commit message: schematic 80%/board 35%
Parts:
- added TP1, TP2: TPPAD1-13, testpad:P1-13
- JP2: device pinhead:1X04 -> pinhead:1X06
- moved JP2 21.4 mm to (47.5, 29.0), turned to 90 degrees
- moved C13 6.94 mm to (11.7, 12.2), turned to 270 degrees
- moved R2 6.90 mm to (7.62, 67.6)
- moved C2 6.27 mm to (11.2, 66.5), turned to 0 degrees
- moved C12 5.86 mm to (34.5, 13.0), turned to 270 degrees
- moved R6 5.09 mm to (19.3, 31.5), turned to 180 degrees
- moved C3 4.23 mm to (7.62, 59.7), turned to 180 degrees
- moved R3 3.54 mm to (10.9, 58.4), turned to 90 degrees
- moved R5 3.06 mm to (14.7, 18.5)
- moved C8 2.81 mm to (7.62, 63.2)
- moved C1 2.17 mm to (13.5, 62.5)
- moved C9 2.05 mm to (33.5, 36.8)
- moved C10 1.27 mm to (33.5, 39.1), turned to 0 degrees
- moved C7 1.14 mm to (17.0, 37.3)
- moved C11 0.92 mm to (13.2, 51.6), turned to 0 degrees
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Connections:
- net N$3 renamed MSG_CG
- net N$36 renamed LAY2_SUPPLY
- net N$37 renamed ATM_RST
- net N$38 renamed CRY_1
- net N$4 renamed MSG_CKIN
- net N$41 renamed CRY_2
- net N$42 renamed LAY3_SUPPLY
- net N$43 renamed LAY4_SUPPLY
- net N$44 renamed MSG_INPUT
- net N$6 renamed UNFILTERED_INPUT
- new net TLC1_ERR: TP2.TP, U2.23
- new net TLC2_ERR: TP1.TP, U3.23
Routing:
- net +5V: track 95.3 -> 179.8 mm, vias 0 -> 2
- net ATM_RST: track 0.00 -> 36.7 mm, vias 0 -> 1
- net SPI_SCLK: track 26.2 -> 55.8 mm, vias 0 -> 2
- net TLC_BLANK: track 0.00 -> 28.1 mm, vias 0 -> 2
- net SPI_MOSI: track 20.4 -> 46.8 mm, vias 2 -> 3
- net MSG_OUT: track 0.00 -> 25.6 mm, vias 0 -> 2
- net N$33: track 0.00 -> 17.9 mm, vias 0 -> 2
- net TLC_VPRG: track 0.00 -> 17.5 mm
- net TLC_GSCLK: track 0.00 -> 16.4 mm
- net N$35: track 0.00 -> 16.3 mm, vias 0 -> 2
- net TLC_XLAT: track 0.00 -> 14.2 mm
- net MSG_INPUT: track 0.00 -> 9.79 mm
- net MSG_CKIN: track 0.00 -> 6.93 mm
- net MSG_CG: track 0.00 -> 4.11 mm
- net N$39: track 0.00 -> 2.72 mm

Commit message: prelim schematic done. second draft of board [50%]
Parts:
- removed C8: 10nF, rcl:C0805
- removed JP4: SUPPLY, pinhead:1X02
- added J1: POWER_JACKPTH, SparkFun-Connectors:POWER_JACK_PTH
- added R7, R8, R9: 1k, rcl:R0805
- added TP3, TP4, TP5, TP6: TPPAD1-13, testpad:P1-13
- C10, C12, C13, C7, C9: value 1uF -> .1uF; device rcl:C0805 -> rcl:C0402
- C11: value 1uF -> .1uF
- C2: value blocking cap -> 10nF
- Q2, Q3, Q4: value (none) -> IRF9530; device transistor-power:TO220BH -> transistor-power:TO220BV
- R4, R5: device rcl:R0805 -> rcl:R0402
- SV1: value (none) -> LED_R; device con-lsta:FE09 -> pinhead:1X09
- SV2: value (none) -> LED_G; device con-lsta:FE09 -> pinhead:1X09
- SV3: value (none) -> LED_B; device con-lsta:FE09 -> pinhead:1X09
- U2, U3: value TLC5940PWP -> TLC5940-RHB; device SparkFun-DigitalIC:TSSOP28-GROUNDPAD -> SparkFun-DigitalIC:QFN-32
- moved SV3 41.0 mm to (45.1, 20.8)
- moved Q3 36.8 mm to (11.8, 61.8), turned to 90 degrees
- moved R1 34.8 mm to (39.1, 64.2), turned to 270 degrees
- moved Q2 34.0 mm to (3.40, 61.7), turned to 90 degrees
- moved C2 32.5 mm to (40.9, 53.4), turned to 270 degrees
- moved R2 32.5 mm to (39.1, 59.7), turned to 90 degrees
- moved C1 32.2 mm to (40.8, 45.5), turned to 90 degrees
- moved X1 31.5 mm to (32.4, 68.8), turned to 0 degrees
- moved JP3 31.4 mm to (30.9, 30.3), turned to 0 degrees
- moved C5 29.5 mm to (25.6, 58.5)
- moved U2 28.9 mm to (13.5, 21.6), turned to 180 degrees
- moved C3 28.2 mm to (34.7, 51.9)
- moved JP1 27.9 mm to (9.40, 71.3)
- moved C6 27.5 mm to (20.4, 57.7), turned to 0 degrees
- moved R3 25.4 mm to (34.6, 49.3), turned to 0 degrees
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Connections:
- net N$13 renamed LED8
- net N$15 renamed LED9
- net N$21 renamed LED23
- net N$22 renamed LED22
- net N$23 renamed LED21
- removed net N$10: SV1.5, U2.11
- removed net N$11: SV1.4, U2.12
- removed net N$12: SV1.3, U2.13
- removed net N$14: SV3.1, U3.17
- removed net N$16: SV3.2, U3.16
- removed net N$17: SV3.3, U3.15
- removed net N$18: SV3.4, U3.14
- removed net N$19: SV3.5, U3.13
- removed net N$20: SV3.6, U3.12
- removed net N$24: SV2.1, U3.8
- removed net N$25: SV2.2, U3.7
- removed net N$26: SV2.9, U2.16
- removed net N$27: SV2.8, U2.17
- removed net N$28: SV2.7, U2.18
- removed net N$29: SV2.6, U2.19
- removed net N$30: SV2.5, U2.20
- removed net N$31: SV2.4, U2.21
- removed net N$32: SV2.3, U2.22
- removed net N$33: JP2.2, U1.30
- removed net N$34: U2.24, U3.5
- removed net N$39: R5.1, U3.27
- removed net N$40: R4.1, U2.27
- removed net N$5: SV1.6, U2.10
- removed net N$7: SV1.9, U2.7
- removed net N$8: SV1.8, U2.8
- removed net N$9: SV1.7, U2.9
- removed net TLC_VPRG: U1.2, U2.6, U3.6
- new net LED1: SV1.9, U2.5
- new net LED11: SV2.9, U2.17
- new net LED12: SV2.8, U2.18
- new net LED13: SV2.7, U2.19
- new net LED14: SV2.6, U2.20
- new net LED15: SV2.5, U2.21
- new net LED16: SV2.4, U3.4
- new net LED17: SV2.3, U3.5
- new net LED18: SV2.2, U3.6
- new net LED19: SV2.1, U3.7
- new net LED2: SV1.8, U2.6
- new net LED24: SV3.6, U3.14
- new net LED25: SV3.5, U3.15
- new net LED26: SV3.4, U3.16
- new net LED27: SV3.3, U3.17
- new net LED28: SV3.2, U3.18
- new net LED29: SV3.1, U3.19
- new net LED3: SV1.7, U2.7
- new net LED4: SV1.6, U2.8
- new net LED5: SV1.5, U2.9
- new net LED6: SV1.4, U2.10
- new net LED7: SV1.3, U2.11
- new net SERIAL_RX: JP2.5, U1.30
- new net TLC1_IREF: R4.1, U2.26
- new net TLC2_IREF: R5.1, U3.26
- new net TLC_CHAIN: U2.23, U3.2
- net +5V: now also J1.PWR, R7.1, R8.1, R9.1, U2.27, U2.3, U3.27, U3.3; no longer JP2.1, JP4.1, U2.28, U3.28
- net ATM_RST: now also TP3.TP
- net GND: now also J1.GND, J1.GNDBREAK, JP2.1, U2.30, U3.30; no longer C8.2, JP2.4, JP4.2, U2.1, U3.1
- net LAYER1_OFF: now also R7.2
- net LAYER2_OFF: now also R9.2
- net LAYER3_OFF: now also R8.2
- net MSG_INPUT: now also TP5.TP
- net MSG_OUT: now also TP6.TP
- net MSG_RST: now also U1.2; no longer U1.13
- net MSG_STROBE: now also U1.32; no longer U1.14
- net N$35: now also JP2.4; no longer JP2.3
- net SPI_MOSI: now also U2.2; no longer U2.5
- net SPI_SCLK: now also U2.1, U3.1; no longer U2.4, U3.4
- net TLC1_ERR: now also U2.22; no longer U2.23
- net TLC2_ERR: now also U3.22; no longer U3.23
- net TLC_BLANK: now also U1.14, U2.31, U3.31; no longer U1.9, U2.2, U3.2
- net TLC_GSCLK: now also U2.24, U3.24; no longer U2.25, U3.25
- net TLC_XLAT: now also U1.13, U2.32, U3.32; no longer U1.32, U2.3
- net UNFILTERED_INPUT: now also TP4.TP; no longer C8.1
Routing:
- net SPI_SCLK: track 55.8 -> 10.3 mm, vias 2 -> 0
- net SPI_MOSI: track 46.8 -> 17.1 mm, vias 3 -> 0
- net SPI_MISO: track 26.7 -> 0.00 mm
- net LAY2_SUPPLY: track 38.9 -> 12.7 mm
- net LED21: track 0.00 -> 25.2 mm
- net LED22: track 0.00 -> 23.7 mm
- net LED23: track 0.00 -> 21.9 mm
- net LED29: track 0.00 -> 21.8 mm
- net LED24: track 0.00 -> 21.5 mm
- net LED25: track 0.00 -> 21.3 mm
- net LED28: track 0.00 -> 21.0 mm
- net LED26: track 0.00 -> 20.9 mm
- net LED27: track 0.00 -> 20.1 mm
- net SERIAL_RX: track 0.00 -> 18.3 mm
- net N$33: track 17.9 -> 0.00 mm, vias 2 -> 0
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