File: LED_Cube.sch (EAGLE design)
At the start: 35 parts, among them IC1 MSGEQ7SOIC, Q1 16MHz, U1 ATMEGA328P-AU, U2 TLC5940PWP, U3 TLC5940PWP, X1 1503_02

Commit message: schematic 80%/board 35%
Parts:
- added TP1, TP2: TPPAD1-13, testpad:TPPAD1-13
- JP2: device pinhead:PINHD-1X4 -> pinhead:PINHD-1X6
Connections:
- net N$3 renamed MSG_CG
- net N$36 renamed LAY2_SUPPLY
- net N$37 renamed ATM_RST
- net N$38 renamed CRY_1
- net N$4 renamed MSG_CKIN
- net N$41 renamed CRY_2
- net N$42 renamed LAY3_SUPPLY
- net N$43 renamed LAY4_SUPPLY
- net N$44 renamed MSG_INPUT
- net N$6 renamed UNFILTERED_INPUT
- new net TLC1_ERR: TP2.TP, U2.XERR
- new net TLC2_ERR: TP1.TP, U3.XERR
Changed lines of the file:
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@@
 <part name="R4" library="rcl" deviceset="R-US_" device="R0805" value="1.9k"/>
 <part name="R5" library="rcl" deviceset="R-US_" device="R0805" value="1.9k"/>
-<part name="JP2" library="pinhead" deviceset="PINHD-1X4" device="" value="SERIAL"/>
+<part name="JP2" library="pinhead" deviceset="PINHD-1X6" device="" value="SERIAL"/>
 <part name="JP3" library="pinhead" deviceset="PINHD-2X3" device="" value="SPI"/>
 <part name="GND6" library="supply1" deviceset="GND" device=""/>
@@
 <part name="GND18" library="supply1" deviceset="GND" device=""/>
 <part name="GND19" library="supply1" deviceset="GND" device=""/>
+<part name="TP1" library="testpad" deviceset="TP" device="PAD1-13"/>
+<part name="TP2" library="testpad" deviceset="TP" device="PAD1-13"/>
 </parts>
 <sheets>
@@
 <instance part="R4" gate="G$1" x="187.96" y="68.58" rot="R270"/>
 <instance part="R5" gate="G$1" x="187.96" y="-12.7" rot="R270"/>
-<instance part="JP2" gate="A" x="106.68" y="81.28"/>
+<instance part="JP2" gate="A" x="109.22" y="81.28"/>
 <instance part="JP3" gate="A" x="114.3" y="134.62"/>
 <instance part="GND6" gate="1" x="129.54" y="127"/>
 <instance part="P+8" gate="1" x="129.54" y="142.24"/>
 <instance part="GND7" gate="1" x="96.52" y="73.66"/>
-<instance part="P+9" gate="1" x="96.52" y="91.44"/>
+<instance part="P+9" gate="1" x="96.52" y="101.6"/>
 <instance part="JP4" gate="G$1" x="-22.86" y="152.4"/>
 <instance part="P+10" gate="1" x="-33.02" y="162.56"/>
@@
 <instance part="GND18" gate="1" x="187.96" y="101.6"/>
 <instance part="GND19" gate="1" x="187.96" y="25.4"/>
+<instance part="TP1" gate="G$1" x="187.96" y="0" rot="R90"/>
+<instance part="TP2" gate="G$1" x="187.96" y="78.74" rot="R90"/>
 </instances>
 <busses>
@@
 <segment>
 <pinref part="JP2" gate="A" pin="1"/>
-<wire x1="104.14" y1="86.36" x2="96.52" y2="86.36" width="0.1524" layer="91"/>
-<wire x1="96.52" y1="86.36" x2="96.52" y2="88.9" width="0.1524" layer="91"/>
+<wire x1="106.68" y1="88.9" x2="96.52" y2="88.9" width="0.1524" layer="91"/>
+<wire x1="96.52" y1="88.9" x2="96.52" y2="99.06" width="0.1524" layer="91"/>
 <pinref part="P+9" gate="1" pin="+5V"/>
 </segment>
@@
 <segment>
 <pinref part="JP2" gate="A" pin="4"/>
-<wire x1="104.14" y1="78.74" x2="96.52" y2="78.74" width="0.1524" layer="91"/>
-<wire x1="96.52" y1="78.74" x2="96.52" y2="76.2" width="0.1524" layer="91"/>
+<wire x1="106.68" y1="81.28" x2="96.52" y2="81.28" width="0.1524" layer="91"/>
+<wire x1="96.52" y1="81.28" x2="96.52" y2="76.2" width="0.1524" layer="91"/>
 <pinref part="GND7" gate="1" pin="GND"/>
 </segment>
@@
 </segment>
 </net>
-<net name="N$6" class="0">
+<net name="UNFILTERED_INPUT" class="0">
 <segment>
 <wire x1="-99.06" y1="114.3" x2="-99.06" y2="121.92" width="0.1524" layer="91"/>
@@
 </segment>
 </net>
-<net name="N$4" class="0">
+<net name="MSG_CKIN" class="0">
 <segment>
 <pinref part="IC1" gate="G$1" pin="CKIN"/>
@@
 </segment>
 </net>
-<net name="N$3" class="0">
+<net name="MSG_CG" class="0">
 <segment>
 <pinref part="C1" gate="G$1" pin="1"/>
@@
 <pinref part="U1" gate="A" pin="PD0"/>
 <wire x1="78.74" y1="71.12" x2="86.36" y2="71.12" width="0.1524" layer="91"/>
-<wire x1="86.36" y1="71.12" x2="86.36" y2="83.82" width="0.1524" layer="91"/>
+<wire x1="86.36" y1="71.12" x2="86.36" y2="86.36" width="0.1524" layer="91"/>
 <pinref part="JP2" gate="A" pin="2"/>
-<wire x1="86.36" y1="83.82" x2="104.14" y2="83.82" width="0.1524" layer="91"/>
+<wire x1="86.36" y1="86.36" x2="106.68" y2="86.36" width="0.1524" layer="91"/>
 </segment>
 </net>
@@
 <pinref part="U1" gate="A" pin="PD1"/>
 <wire x1="78.74" y1="68.58" x2="88.9" y2="68.58" width="0.1524" layer="91"/>
-<wire x1="88.9" y1="68.58" x2="88.9" y2="81.28" width="0.1524" layer="91"/>
+<wire x1="88.9" y1="68.58" x2="88.9" y2="83.82" width="0.1524" layer="91"/>
 <pinref part="JP2" gate="A" pin="3"/>
-<wire x1="88.9" y1="81.28" x2="104.14" y2="81.28" width="0.1524" layer="91"/>
+<wire x1="88.9" y1="83.82" x2="106.68" y2="83.82" width="0.1524" layer="91"/>
 </segment>
 </net>
@@
 </segment>
 </net>
-<net name="N$37" class="0">
+<net name="ATM_RST" class="0">
 <segment>
 <pinref part="U1" gate="A" pin="PC6"/>
@@
 </segment>
 </net>
-<net name="N$38" class="0">
+<net name="CRY_1" class="0">
 <segment>
 <pinref part="U1" gate="A" pin="PB6"/>
@@
 </segment>
 </net>
-<net name="N$41" class="0">
+<net name="CRY_2" class="0">
 <segment>
 <pinref part="U1" gate="A" pin="PB7"/>
@@
 </segment>
 </net>
-<net name="N$36" class="0">
+<net name="LAY2_SUPPLY" class="0">
 <segment>
 <pinref part="Q3" gate="G$1" pin="D"/>
@@
 </segment>
 </net>
-<net name="N$42" class="0">
+<net name="LAY3_SUPPLY" class="0">
 <segment>
 <pinref part="JP1" gate="A" pin="2"/>
@@
 </segment>
 </net>
-<net name="N$43" class="0">
+<net name="LAY4_SUPPLY" class="0">
 <segment>
 <pinref part="JP1" gate="A" pin="1"/>
@@
 </segment>
 </net>
-<net name="N$44" class="0">
+<net name="MSG_INPUT" class="0">
 <segment>
 <pinref part="C2" gate="G$1" pin="2"/>
@@
 </segment>
 </net>
+<net name="TLC1_ERR" class="0">
+<segment>
+<pinref part="U2" gate="G$1" pin="XERR"/>
+<pinref part="TP2" gate="G$1" pin="TP"/>
+<wire x1="200.66" y1="78.74" x2="190.5" y2="78.74" width="0.1524" layer="91"/>
+</segment>
+</net>
+<net name="TLC2_ERR" class="0">
+<segment>
+<pinref part="U3" gate="G$1" pin="XERR"/>
+<pinref part="TP1" gate="G$1" pin="TP"/>
+<wire x1="200.66" y1="0" x2="190.5" y2="0" width="0.1524" layer="91"/>
+</segment>
+</net>

Commit message: prelim schematic done. second draft of board [50%]
Parts:
- removed C8: 10nF, rcl:C-EUC0805
- removed JP4: SUPPLY, pinhead:PINHD-1X2
- added J1: POWER_JACKPTH, SparkFun-Connectors:POWER_JACKPTH
- added R7, R8, R9: 1k, rcl:R-US_R0805
- added TP3, TP4, TP5, TP6: TPPAD1-13, testpad:TPPAD1-13
- C10, C12, C13, C7, C9: value 1uF -> .1uF; device rcl:C-EUC0805 -> rcl:C-EUC0402
- C11: value 1uF -> .1uF
- C2: value blocking cap -> 10nF
- Q2, Q3, Q4: value (none) -> IRF9530; device transistor-power:PMOSFET_PTO220BH -> transistor-power:IRF9530
- R4, R5: device rcl:R-US_R0805 -> rcl:R-US_R0402
- SV1: value (none) -> LED_R; device con-lsta:FE09-1 -> pinhead:PINHD-1X9
- SV2: value (none) -> LED_G; device con-lsta:FE09-1 -> pinhead:PINHD-1X9
- SV3: value (none) -> LED_B; device con-lsta:FE09-1 -> pinhead:PINHD-1X9
- U2, U3: value TLC5940PWP -> TLC5940-RHB; device SparkFun-DigitalIC:TLC5940PWP -> SparkFun-DigitalIC:TLC5940-RHB
Connections:
- net N$34 renamed TLC_CHAIN
- net N$39 renamed TLC2_IREF
- net N$40 renamed TLC1_IREF
- removed net N$10: SV1.5, U2.OUT4
- removed net N$11: SV1.4, U2.OUT5
- removed net N$12: SV1.3, U2.OUT6
- removed net N$13: SV1.2, U2.OUT7
- removed net N$14: SV3.1, U3.OUT10
- removed net N$15: SV1.1, U2.OUT8
- removed net N$16: SV3.2, U3.OUT9
- removed net N$17: SV3.3, U3.OUT8
- removed net N$18: SV3.4, U3.OUT7
- removed net N$19: SV3.5, U3.OUT6
- removed net N$20: SV3.6, U3.OUT5
- removed net N$21: SV3.7, U3.OUT4
- removed net N$22: SV3.8, U3.OUT3
- removed net N$23: SV3.9, U3.OUT2
- removed net N$24: SV2.1, U3.OUT1
- removed net N$25: SV2.2, U3.OUT0
- removed net N$26: SV2.9, U2.OUT9
- removed net N$27: SV2.8, U2.OUT10
- removed net N$28: SV2.7, U2.OUT11
- removed net N$29: SV2.6, U2.OUT12
- removed net N$30: SV2.5, U2.OUT13
- removed net N$31: SV2.4, U2.OUT14
- removed net N$32: SV2.3, U2.OUT15
- removed net N$33: JP2.2, U1.PD0
- removed net N$5: SV1.6, U2.OUT3
- removed net N$7: SV1.9, U2.OUT0
- removed net N$8: SV1.8, U2.OUT1
- removed net N$9: SV1.7, U2.OUT2
- removed net TLC_VPRG: U1.PD4, U2.VPRG, U3.VPRG
- new net LED1: SV1.9, U2.OUT1
- new net LED11: SV2.9, U2.OUT11
- new net LED12: SV2.8, U2.OUT12
- new net LED13: SV2.7, U2.OUT13
- new net LED14: SV2.6, U2.OUT14
- new net LED15: SV2.5, U2.OUT15
- new net LED16: SV2.4, U3.OUT0
- new net LED17: SV2.3, U3.OUT1
- new net LED18: SV2.2, U3.OUT2
- new net LED19: SV2.1, U3.OUT3
- new net LED2: SV1.8, U2.OUT2
- new net LED21: SV3.9, U3.OUT5
- new net LED22: SV3.8, U3.OUT6
- new net LED23: SV3.7, U3.OUT7
- new net LED24: SV3.6, U3.OUT8
- new net LED25: SV3.5, U3.OUT9
- new net LED26: SV3.4, U3.OUT10
- new net LED27: SV3.3, U3.OUT11
- new net LED28: SV3.2, U3.OUT12
- new net LED29: SV3.1, U3.OUT13
- new net LED3: SV1.7, U2.OUT3
- new net LED4: SV1.6, U2.OUT4
- new net LED5: SV1.5, U2.OUT5
- new net LED6: SV1.4, U2.OUT6
- new net LED7: SV1.3, U2.OUT7
- new net LED8: SV1.2, U2.OUT8
- new net LED9: SV1.1, U2.OUT9
- new net SERIAL_RX: JP2.5, U1.PD0
- net +5V: now also J1.PWR, R7.1, R8.1, R9.1, U2.VPRG, U3.VPRG; no longer JP2.1, JP4.1
- net ATM_RST: now also TP3.TP
- net GND: now also J1.GND, J1.GNDBREAK, JP2.1; no longer C8.2, JP2.4, JP4.2
- net LAYER1_OFF: now also R7.2
- net LAYER2_OFF: now also R9.2
- net LAYER3_OFF: now also R8.2
- net MSG_INPUT: now also TP5.TP
- net MSG_OUT: now also TP6.TP
- net MSG_RST: now also U1.PD4; no longer U1.PB1
- net MSG_STROBE: now also U1.PD2; no longer U1.PB2
- net N$35: now also JP2.4; no longer JP2.3
- net TLC_BLANK: now also U1.PB2; no longer U1.PD5
- net TLC_XLAT: now also U1.PB1, U3.XLAT; no longer U1.PD2
- net UNFILTERED_INPUT: now also TP4.TP; no longer C8.1
Other:
- moved on the sheet: C1, C10, C11, C12, C13, C2, C3, C4, C5, C6, C7, C9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
