File: T02_LED_Cube.brd (EAGLE design)
At the start: 61.9 x 80 mm, 43 parts, among them IC1 MSGEQ7SOIC, J1 POWER_JACKPTH, Q1 16MHz, Q2 IRF9530, Q3 IRF9530, Q4 IRF9530, U1 ATMEGA328P-AU, U2 TLC5940-RHB, U3 TLC5940-RHB, X1 1503_02

Commit message: pcb 75% done
Parts:
- added R10: 0, rcl:R1210
- C10, C12, C13, C7, C9: value .1uF -> .15uF
- C11: value .1uF -> .15uF; device rcl:C0805 -> rcl:C0402
- moved C5 11.1 mm to (21.3, 48.3)
- moved TP3 10.8 mm to (44.9, 32.7)
- moved C2 7.60 mm to (44.7, 60.0)
- moved C1 6.55 mm to (42.6, 51.8)
- moved R3 6.28 mm to (36.2, 55.4)
- moved C12 6.19 mm to (18.1, 22.0)
- moved IC1 5.90 mm to (37.1, 50.8)
- moved C3 5.79 mm to (36.3, 57.5)
- moved Q3 5.47 mm to (17.1, 63.0)
- moved JP3 5.44 mm to (36.3, 30.2)
- moved TP5 5.38 mm to (42.5, 46.2)
- moved C11 5.21 mm to (32.3, 52.0), turned to 270 degrees
- moved Q1 4.83 mm to (25.5, 53.2), turned to 90 degrees
- moved JP1 4.75 mm to (4.83, 70.1)
- moved TP4 4.58 mm to (47.3, 62.9)
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Connections:
- net LAY4_SUPPLY renamed LAY1_SUPPLY
- net N$35 renamed SERIAL_TX
- new net LED_SUPPLY: Q2.S, Q3.S, Q4.S, R10.1, R7.1, R8.1, R9.1
- net +5V: now also R10.2; no longer Q2.S, Q3.S, Q4.S, R7.1, R8.1, R9.1
Routing:
- net TLC_GSCLK: track 19.4 -> 53.9 mm, vias 2 -> 3
- net +5V: track 170.9 -> 140.6 mm, vias 4 -> 2
- net SPI_SCLK: track 10.3 -> 37.4 mm, vias 0 -> 2
- net TLC_XLAT: track 9.57 -> 33.6 mm, vias 2 -> 3
- net SPI_MISO: track 0.00 -> 21.8 mm, vias 0 -> 1
- net SPI_MOSI: track 17.1 -> 34.4 mm, vias 0 -> 1
- net UNFILTERED_INPUT: track 14.5 -> 0.00 mm
- net N$2: track 11.8 -> 0.00 mm
- net MSG_STROBE: track 4.31 -> 13.2 mm
- net LAY3_SUPPLY: track 18.7 -> 10.7 mm
- net ATM_RST: track 19.5 -> 26.7 mm
- net MSG_OUT: track 21.5 -> 27.7 mm, vias 2 -> 1
- net LED14: track 8.69 -> 14.8 mm
- net CRY_2: track 18.5 -> 23.8 mm
- net CRY_1: track 16.2 -> 11.8 mm
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Other:
- board size 61.9 x 80 mm -> 50.5 x 66.8 mm

Commit message: board 95% besides stitching
Parts:
- moved R2 3.17 mm to (38.4, 62.0)
- moved X1 1.60 mm to (30.8, 72.6)
- moved C2 0.95 mm to (44.5, 61.0)
- moved TP6 0.92 mm to (31.8, 47.2)
- moved R1 0.63 mm to (42.2, 64.8)
- moved R7 0.51 mm to (12.4, 50.8)
Routing:
- net LED_SUPPLY: track 0.00 -> 49.5 mm
- net N$2: track 0.00 -> 18.0 mm
- net UNFILTERED_INPUT: track 0.00 -> 10.4 mm
- net LAYER2_OFF: track 26.3 -> 30.7 mm
- net LAYER1_OFF: track 17.1 -> 21.1 mm
- net +5V: track 140.6 -> 137.1 mm, vias 2 -> 1
- net LAYER3_OFF: track 27.8 -> 31.0 mm
- net N$1: track 0.00 -> 2.93 mm
- net MSG_OUT: track 27.7 -> 25.7 mm
- net MSG_INPUT: track 17.3 -> 18.1 mm
Other:
- board size 50.5 x 66.8 mm -> 50.2 x 66.5 mm

Commit message: submitted board
Parts:
- removed C13: .15uF, rcl:C0402
- removed SV1: LED_R, pinhead:1X09
- added C8: .15uF, rcl:C0402
- added JP6: LED_SUPPLY, pinhead:1X03
- added R11, R12, R13, R14: 0, rcl:R0402
- C1: value .1uF -> 10nF
- C10: value .15uF -> 33pF; device rcl:C0402 -> rcl:C0805
- C2: value 10nF -> .15uF; device rcl:C0805 -> rcl:C0402
- C3: value 33pF -> 1uF
- C4: value 1uF -> .15uF; device rcl:C0805 -> rcl:C0402
- C6: value 22pF -> .15uF; device rcl:C0805 -> rcl:C0402
- C7: value .15uF -> .1uF; device rcl:C0402 -> rcl:C0805
- C9: value .15uF -> 22pF; device rcl:C0402 -> rcl:C0805
- JP1: value LED_SUPPLY -> SPI; device pinhead:1X03 -> pinhead:2X03
- JP3: value SPI -> LED_R; device pinhead:2X03 -> pinhead:1X09
- R10: value 0 -> 1k; device rcl:R1210 -> rcl:R0805
- R4: value 1.9k -> 4.7k; device rcl:R0402 -> rcl:R0805
- R5: value 1.9k -> 1k; device rcl:R0402 -> rcl:R0805
- R6: value 4.7k -> 1.9k; device rcl:R0805 -> rcl:R0402
- R7: value 1k -> 1.9k; device rcl:R0805 -> rcl:R0402
- R9: value 1k -> 0; device rcl:R0805 -> rcl:R1210
- moved JP1 50.8 mm to (36.3, 30.2)
- moved JP3 34.9 mm to (2.64, 21.1), turned to 90 degrees
- moved C11 33.2 mm to (18.1, 22.0), turned to 90 degrees
- moved C3 32.9 mm to (12.4, 34.8), turned to 270 degrees
- moved R5 31.4 mm to (12.4, 50.8), turned to 270 degrees
- moved R7 31.4 mm to (30.9, 25.3), turned to 90 degrees
- moved C7 27.6 mm to (42.6, 51.8), turned to 90 degrees
- moved R4 20.3 mm to (31.8, 35.1), turned to 270 degrees
- moved R10 19.6 mm to (22.9, 62.9), flipped to the top
- moved R9 19.6 mm to (15.0, 45.0), flipped to the bottom
- moved R6 19.5 mm to (18.3, 20.3), turned to 0 degrees
- moved C10 19.1 mm to (36.3, 57.5), turned to 180 degrees
- moved Q4 16.1 mm to (17.1, 63.0)
- moved C2 15.1 mm to (32.3, 52.0)
- moved C9 12.6 mm to (21.3, 55.4), turned to 270 degrees
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- renumbered SV2 to JP4, SV3 to JP5
Connections:
- new net N$3: R12.2, U3.3
- new net N$4: R14.2, U2.3
- new net N$5: R11.2, U3.25
- new net N$6: R13.2, U2.25
- net +5V: now also C2.1, C3.1, C6.1, C8.1, JP1.2, R11.1, R12.1, R13.1, R14.1, R4.2, R9.2; no longer C10.1, C13.1, C7.1, C9.1, JP3.2, R10.2, R6.2, U2.3, U3.3
- net ATM_RST: now also JP1.5, R4.1; no longer JP3.5, R6.1
- net CRY_2: now also C9.1; no longer C6.1
- net GND: now also C2.2, C8.2, JP1.6, R6.2, R7.2; no longer C1.2, C13.2, JP3.6, R4.2, R5.2
- net LAY1_SUPPLY: now also JP6.1, Q2.D; no longer JP1.1, Q4.D
- net LAY2_SUPPLY: now also JP6.3, Q4.D; no longer JP1.3, Q3.D
- net LAY3_SUPPLY: now also JP6.2, Q3.D; no longer JP1.2, Q2.D
- net LAYER1_OFF: now also Q2.G, R5.2; no longer Q4.G, R7.2
- net LAYER2_OFF: now also Q4.G, R10.2; no longer Q3.G, R9.2
- net LAYER3_OFF: now also Q3.G; no longer Q2.G
- net LED1: now also JP3.9; no longer SV1.9
- net LED2: now also JP3.8; no longer SV1.8
- net LED3: now also JP3.7; no longer SV1.7
- net LED4: now also JP3.6; no longer SV1.6
- net LED5: now also JP3.5; no longer SV1.5
- net LED6: now also JP3.4; no longer SV1.4
- net LED7: now also JP3.3; no longer SV1.3
- net LED8: now also JP3.2; no longer SV1.2
- net LED9: now also JP3.1; no longer SV1.1
- net LED_SUPPLY: now also R5.1; no longer R7.1
- net MSG_CG: now also C7.1; no longer C1.1
- net MSG_CKIN: now also C10.1; no longer C3.1
- net MSG_INPUT: now also C1.2; no longer C2.2
- net SPI_MISO: now also JP1.1; no longer JP3.1
- net SPI_MOSI: now also JP1.4; no longer JP3.4
- net SPI_SCLK: now also JP1.3; no longer JP3.3
- net TLC1_IREF: now also R6.1; no longer R4.1
- net TLC2_IREF: now also R7.1; no longer R5.1
- net UNFILTERED_INPUT: now also C1.1; no longer C2.1
Routing:
- net GND: track 0.00 -> 8.47 mm, vias 0 -> 14
- net N$5: track 0.00 -> 6.16 mm
- net N$3: track 0.00 -> 3.84 mm
- net N$6: track 0.00 -> 2.03 mm
- net N$4: track 0.00 -> 1.78 mm
- net TLC_GSCLK: track 53.9 -> 54.8 mm
- net +5V: track 137.1 -> 136.5 mm
- net TLC_CHAIN: track 15.2 -> 15.8 mm
- added copper zone on layer 16, net GND
Other:
- board size 50.2 x 66.5 mm -> 50 x 66.5 mm
- board text added: "1"
- board text added: "11"
- board text added: "19"
- board text added: "21"
- board text added: "29"
- board text added: "9"
- board text added: "BLUE"
- board text added: "GREEN"
- board text added: "ICSP/SPI"
- board text added: "LED-Cube 2016 Practicum T02 Evan Yand, Matthew Konyndyk, Jasjit Singh, Alex Mendez"
- board text added: "RED"
- board text added: "RX"
- board text added: "TX"
