File: T02_LED_Cube.sch (EAGLE design)
At the start: 43 parts, among them IC1 MSGEQ7SOIC, J1 POWER_JACKPTH, Q1 16MHz, Q2 IRF9530, Q3 IRF9530, Q4 IRF9530, U1 ATMEGA328P-AU, U2 TLC5940-RHB, U3 TLC5940-RHB, X1 1503_02

Commit message: pcb 75% done
Parts:
- added R10: 0, rcl:R-US_R1210
- C10, C12, C13, C7, C9: value .1uF -> .15uF
- C11: value .1uF -> .15uF; device rcl:C-EUC0805 -> rcl:C-EUC0402
Connections:
- net LAY4_SUPPLY renamed LAY1_SUPPLY
- net N$35 renamed SERIAL_TX
- new net LED_SUPPLY: Q2.S, Q3.S, Q4.S, R10.1, R7.1, R8.1, R9.1
- net +5V: now also R10.2; no longer Q2.S, Q3.S, Q4.S, R7.1, R8.1, R9.1
Other:
- moved on the sheet: JP1, Q2, Q3, Q4, R7, R8, R9

Commit message: submitted board
Parts:
- removed C13: .15uF, rcl:C-EUC0402
- removed SV1: LED_R, pinhead:PINHD-1X9
- added C8: .15uF, rcl:C-EUC0402
- added JP6: LED_SUPPLY, pinhead:PINHD-1X3
- added R11, R12, R13, R14: 0, rcl:R-US_R0402
- C1: value .1uF -> 10nF
- C10: value .15uF -> 33pF; device rcl:C-EUC0402 -> rcl:C-EUC0805
- C2: value 10nF -> .15uF; device rcl:C-EUC0805 -> rcl:C-EUC0402
- C3: value 33pF -> 1uF
- C4: value 1uF -> .15uF; device rcl:C-EUC0805 -> rcl:C-EUC0402
- C6: value 22pF -> .15uF; device rcl:C-EUC0805 -> rcl:C-EUC0402
- C7: value .15uF -> .1uF; device rcl:C-EUC0402 -> rcl:C-EUC0805
- C9: value .15uF -> 22pF; device rcl:C-EUC0402 -> rcl:C-EUC0805
- JP1: value LED_SUPPLY -> SPI; device pinhead:PINHD-1X3 -> pinhead:PINHD-2X3
- JP3: value SPI -> LED_R; device pinhead:PINHD-2X3 -> pinhead:PINHD-1X9
- R10: value 0 -> 1k; device rcl:R-US_R1210 -> rcl:R-US_R0805
- R4: value 1.9k -> 4.7k; device rcl:R-US_R0402 -> rcl:R-US_R0805
- R5: value 1.9k -> 1k; device rcl:R-US_R0402 -> rcl:R-US_R0805
- R6: value 4.7k -> 1.9k; device rcl:R-US_R0805 -> rcl:R-US_R0402
- R7: value 1k -> 1.9k; device rcl:R-US_R0805 -> rcl:R-US_R0402
- R9: value 1k -> 0; device rcl:R-US_R0805 -> rcl:R-US_R1210
- renumbered SV2 to JP4, SV3 to JP5
Connections:
- new net N$3: R12.2, U3.VPRG
- new net N$4: R14.2, U2.VPRG
- new net N$5: R11.2, U3.DCPRG
- new net N$6: R13.2, U2.DCPRG
- net +5V: now also C2.1, C3.1, C6.1, C8.1, JP1.2, R11.1, R12.1, R13.1, R14.1, R4.2, R9.2; no longer C10.1, C13.1, C7.1, C9.1, JP3.2, R10.2, R6.2, U2.VPRG, U3.VPRG
- net ATM_RST: now also JP1.5, R4.1; no longer JP3.5, R6.1
- net CRY_2: now also C9.1; no longer C6.1
- net GND: now also C2.2, C8.2, JP1.6, R6.2, R7.2; no longer C1.2, C13.2, JP3.6, R4.2, R5.2
- net LAY1_SUPPLY: now also JP6.1, Q2.D; no longer JP1.1, Q4.D
- net LAY2_SUPPLY: now also JP6.3, Q4.D; no longer JP1.3, Q3.D
- net LAY3_SUPPLY: now also JP6.2, Q3.D; no longer JP1.2, Q2.D
- net LAYER1_OFF: now also Q2.G, R5.2; no longer Q4.G, R7.2
- net LAYER2_OFF: now also Q4.G, R10.2; no longer Q3.G, R9.2
- net LAYER3_OFF: now also Q3.G; no longer Q2.G
- net LED1: now also JP3.9; no longer SV1.9
- net LED2: now also JP3.8; no longer SV1.8
- net LED3: now also JP3.7; no longer SV1.7
- net LED4: now also JP3.6; no longer SV1.6
- net LED5: now also JP3.5; no longer SV1.5
- net LED6: now also JP3.4; no longer SV1.4
- net LED7: now also JP3.3; no longer SV1.3
- net LED8: now also JP3.2; no longer SV1.2
- net LED9: now also JP3.1; no longer SV1.1
- net LED_SUPPLY: now also R5.1; no longer R7.1
- net MSG_CG: now also C7.1; no longer C1.1
- net MSG_CKIN: now also C10.1; no longer C3.1
- net MSG_INPUT: now also C1.2; no longer C2.2
- net SPI_MISO: now also JP1.1; no longer JP3.1
- net SPI_MOSI: now also JP1.4; no longer JP3.4
- net SPI_SCLK: now also JP1.3; no longer JP3.3
- net TLC1_IREF: now also R6.1; no longer R4.1
- net TLC2_IREF: now also R7.1; no longer R5.1
- net UNFILTERED_INPUT: now also C1.1; no longer C2.1
Other:
- moved on the sheet: C1, C10, C11, C12, C2, C3, C4, C6, C7, C9, Q2, Q3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
